File: Hardware/Tube Board/CNIX V2 Tube Board/CNIX V2 Tube Board.kicad_sch (KiCad schematic)
At the start: 50 parts, among them J1 VDD, J2 GND, J3 Tube Conn, J4 LED, J5 HT, U1 SN75468, U10 IN-4_0, U11 IN-4_1, U12 IN-4_2, U13 IN-4_3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

Commit message: finished wiring fix for the tube board
Parts:
- U10, U11, U12, U13: footprint .Nixie Tubes:IN-4 -> Nixie_Tubes:IN-4
Connections:
- net T0_D0: now also U14.5 (I5); no longer U14.6 (I6)
- net T0_D1: now also U14.1 (I1); no longer U1.7 (I7)
- net T0_D2: now also U14.4 (I4); no longer U14.7 (I7)
- net T0_D3: now also U14.3 (I3); no longer U1.5 (I5)
- net T0_D4: now also U1.7 (I7); no longer U14.1 (I1)
- net T0_D5: now also U14.2 (I2); no longer U1.6 (I6)
- net T0_D6: now also U1.6 (I6); no longer U14.2 (I2)
- net T0_D7: now also U14.6 (I6); no longer U14.5 (I5)
- net T0_D8: now also U1.5 (I5); no longer U14.3 (I3)
- net T0_D9: now also U14.7 (I7); no longer U14.4 (I4)
- net T0_K0: now also U14.12 (O5); no longer U14.11 (O6)
- net T0_K1: now also U14.16 (O1); no longer U1.10 (O7)
- net T0_K2: now also U14.13 (O4); no longer U14.10 (O7)
- net T0_K3: now also U14.14 (O3); no longer U1.12 (O5)
- net T0_K4: now also U1.10 (O7); no longer U14.16 (O1)
- net T0_K5: now also U14.15 (O2); no longer U1.11 (O6)
- net T0_K6: now also U1.11 (O6); no longer U14.15 (O2)
- net T0_K7: now also U14.11 (O6); no longer U14.12 (O5)
- net T0_K8: now also U1.12 (O5); no longer U14.14 (O3)
- net T0_K9: now also U14.10 (O7); no longer U14.13 (O4)
- net T1_D1: now also U1.1 (I1); no longer U2.6 (I6)
- net T1_D2: now also U1.4 (I4); no longer U2.3 (I3)
- net T1_D3: now also U1.3 (I3); no longer U2.4 (I4)
- net T1_D4: now also U2.7 (I7); no longer U1.1 (I1)
- net T1_D5: now also U1.2 (I2); no longer U2.5 (I5)
- net T1_D6: now also U2.6 (I6); no longer U1.2 (I2)
- net T1_D7: now also U2.3 (I3); no longer U2.1 (I1)
- net T1_D8: now also U2.5 (I5); no longer U1.3 (I3)
- net T1_D9: now also U2.4 (I4); no longer U1.4 (I4)
- net T1_K1: now also U1.16 (O1); no longer U2.11 (O6)
- net T1_K2: now also U1.13 (O4); no longer U2.14 (O3)
- net T1_K3: now also U1.14 (O3); no longer U2.13 (O4)
- net T1_K4: now also U2.10 (O7); no longer U1.16 (O1)
- net T1_K5: now also U1.15 (O2); no longer U2.12 (O5)
- net T1_K6: now also U2.11 (O6); no longer U1.15 (O2)
- net T1_K7: now also U2.14 (O3); no longer U2.16 (O1)
- net T1_K8: now also U2.12 (O5); no longer U1.14 (O3)
- net T1_K9: now also U2.13 (O4); no longer U1.13 (O4)
- net T2_D0: now also U3.5 (I5); no longer U3.6 (I6)
- net T2_D1: now also U3.1 (I1); no longer U4.7 (I7)
- net T2_D2: now also U3.4 (I4); no longer U4.4 (I4)
- net T2_D3: now also U3.3 (I3); no longer U4.5 (I5)
- net T2_D4: now also U4.7 (I7); no longer U3.1 (I1)
- net T2_D5: now also U3.2 (I2); no longer U4.6 (I6)
- net T2_D6: now also U4.6 (I6); no longer U3.2 (I2)
- net T2_D7: now also U3.6 (I6); no longer U3.5 (I5)
- net T2_D8: now also U4.5 (I5); no longer U3.3 (I3)
- net T2_D9: now also U4.4 (I4); no longer U3.4 (I4)
- net T2_K0: now also U3.12 (O5); no longer U3.11 (O6)
- net T2_K1: now also U3.16 (O1); no longer U4.10 (O7)
- net T2_K2: now also U3.13 (O4); no longer U4.13 (O4)
- net T2_K3: now also U3.14 (O3); no longer U4.12 (O5)
- net T2_K4: now also U4.10 (O7); no longer U3.16 (O1)
- net T2_K5: now also U3.15 (O2); no longer U4.11 (O6)
- net T2_K6: now also U4.11 (O6); no longer U3.15 (O2)
- net T2_K7: now also U3.11 (O6); no longer U3.12 (O5)
- net T2_K8: now also U4.12 (O5); no longer U3.14 (O3)
- net T2_K9: now also U4.13 (O4); no longer U3.13 (O4)
- net T3_D0: now also U5.2 (I2); no longer U5.3 (I3)
- net T3_D1: now also U4.1 (I1); no longer U5.7 (I7)
- net T3_D2: now also U5.1 (I1); no longer U5.4 (I4)
- net T3_D3: now also U4.3 (I3); no longer U5.5 (I5)
- net T3_D4: now also U5.7 (I7); no longer U4.1 (I1)
- net T3_D5: now also U4.2 (I2); no longer U5.6 (I6)
- net T3_D6: now also U5.6 (I6); no longer U4.2 (I2)
- net T3_D7: now also U5.3 (I3); no longer U5.2 (I2)
- net T3_D8: now also U5.5 (I5); no longer U4.3 (I3)
- net T3_D9: now also U5.4 (I4); no longer U5.1 (I1)
- net T3_K0: now also U5.15 (O2); no longer U5.14 (O3)
- net T3_K1: now also U4.16 (O1); no longer U5.10 (O7)
- net T3_K2: now also U5.16 (O1); no longer U5.13 (O4)
- net T3_K3: now also U4.14 (O3); no longer U5.12 (O5)
- net T3_K4: now also U5.10 (O7); no longer U4.16 (O1)
- net T3_K5: now also U4.15 (O2); no longer U5.11 (O6)
- net T3_K6: now also U5.11 (O6); no longer U4.15 (O2)
- net T3_K7: now also U5.14 (O3); no longer U5.15 (O2)
- net T3_K8: now also U5.12 (O5); no longer U4.14 (O3)
- net T3_K9: now also U5.13 (O4); no longer U5.16 (O1)
